Commit message: Add simulation evaluation framework, specs and Nav2/SLAM pipeline fixes
- vacuum_eval package: ground truth, odometry noise, recorder, episode
  runner/batch, compute_metrics, aggregate, and offline metric modules
  (coverage, completeness, ATE/RPE, navigation, safety, responsiveness,
  loop closure, cleaning efficiency, resources); 87 unit tests.
- docs/specs: implementation specs for every metric, METRICS_TO_BE_MEASURED,
  HANDOFF and PROJECT_STATUS.
- 14 new/fixed evaluation worlds (corridor sealed, avoid_* scenarios).
- Fixes found by running the stack: Nav2 commands now reach the controller,
  velocity smoother loop, depthimage_to_laserscan remaps (scan was empty),
  navigate.xml invalid Wait port, RTAB-Map topic names and start-up
  deadlock, exploration manager (oscillation, stale results, goal snapping,
  blacklist, finish signal), delete_db, CycloneDDS buffer requirement,
  vacuum_description CMake install error, 4 ms physics step.

Co-Authored-By: Claude Sonnet 5.5 <noreply@anthropic.com>

File: Navigation/Simulation/vacuum_ws/src/vacuum_description/urdf/_gazebo.xacro (robot description, xacro)
@@ -95,4 +95,18 @@
       -->
       <parameters>$(find vacuum_controller)/config/controllers.yaml</parameters>
+    </plugin>
+  </gazebo>
+  <!-- Ground truth for evaluation (docs/specs/01 section 1.1b): the ros_gz_bridge
+       Pose_V -> TFMessage conversion drops entity names, so the robot's true pose
+       is published by this plugin instead. Read by ground_truth_node. -->
+  <gazebo>
+    <plugin filename="gz-sim-odometry-publisher-system"
+            name="gz::sim::systems::OdometryPublisher">
+      <odom_frame>world</odom_frame>
+      <robot_base_frame>base_footprint</robot_base_frame>
+      <odom_topic>/model/vacuum_robot/ground_truth_odom</odom_topic>
+      <odom_publish_frequency>30</odom_publish_frequency>
+      <dimensions>2</dimensions>
+      <gaussian_noise>0</gaussian_noise>
     </plugin>
   </gazebo>
@@ -183,3 +197,30 @@
     </sensor>
   </gazebo>
+  <!-- Contact sensors (spec 06 6.2): body collisions only, not wheels/caster. Names are post-lumping. -->
+  <gazebo reference="base_footprint">
+    <sensor name="chassis_contact" type="contact">
+      <always_on>true</always_on>
+      <update_rate>50</update_rate>
+      <contact>
+        <collision>base_footprint_fixed_joint_lump__base_link_collision</collision>
+        <topic>/vacuum_robot/contacts/chassis</topic>
+      </contact>
+    </sensor>
+    <sensor name="camera_mount_contact" type="contact">
+      <always_on>true</always_on>
+      <update_rate>50</update_rate>
+      <contact>
+        <collision>base_footprint_fixed_joint_lump__camera_mount_link_collision_2</collision>
+        <topic>/vacuum_robot/contacts/camera_mount</topic>
+      </contact>
+    </sensor>
+    <sensor name="camera_contact" type="contact">
+      <always_on>true</always_on>
+      <update_rate>50</update_rate>
+      <contact>
+        <collision>base_footprint_fixed_joint_lump__camera_link_collision_3</collision>
+        <topic>/vacuum_robot/contacts/camera</topic>
+      </contact>
+    </sensor>
+  </gazebo>
 </robot>
